File: Exercise 2.kicad_sch (KiCad schematic)
At the start: 10 parts, among them J1 Conn_01x02_Male, U1 1

Commit message: Add files via upload
Parts:
- removed C1: 10uF, symbol Device:C_Polarized
- added C1: 10uF, Capacitor_Tantalum_SMD:CP_EIA-3216-18_Kemet-A_Pad1.58x1.35mm_HandSolder, symbol Device:C_Polarized_Small
- C2: footprint (none) -> Capacitor_SMD:C_0805_2012Metric_Pad1.18x1.45mm_HandSolder
- D1, D2: footprint (none) -> LED_SMD:LED_1206_3216Metric_Pad1.42x1.75mm_HandSolder
- J1: footprint (none) -> TerminalBlock:TerminalBlock_bornier-2_P5.08mm
- R1: renamed from R3; footprint (none) -> Resistor_SMD:R_0805_2012Metric_Pad1.20x1.40mm_HandSolder
- R2: renamed from R4; value 1k -> 10k; footprint (none) -> Resistor_SMD:R_0805_2012Metric_Pad1.20x1.40mm_HandSolder
- R3: renamed from R1; value 10k -> 1k; footprint (none) -> Resistor_SMD:R_0805_2012Metric_Pad1.20x1.40mm_HandSolder
- R4: renamed from R2; value 10k -> 1k; footprint (none) -> Resistor_SMD:R_0805_2012Metric_Pad1.20x1.40mm_HandSolder
- U1: footprint Package_SO:SOIC-8_3.9x4.9mm_P1.27mm -> Package_SO:SOIC-8-1EP_3.9x4.9mm_P1.27mm_EP2.29x3mm
Connections:
- net 9V is gone; now on net +9V: U1.4 (R)
- net +9V: now also R1.1; no longer R3.1
- net GND: now also C1.2
- net pin_2: now also R2.2, C1.1; no longer R4.2
- net pin_3: now also R3.2, R4.1; no longer R1.2, R2.1
- net at D2.2 (A): now also R4.2; no longer R2.2
- net at D1.1 (K): now also R3.1; no longer R1.1
- new net pin_7: R1.2, R2.1, U1.7 (DIS)
Other:
- note removed: "pin_3"
